File: STM32F103C8T6_FOC.kicad_pcb (KiCad board)
At the start: 2 copper layers, 89 parts, among them IC1 BD9E303EFJ-LBE2, IC2 AS5600-ASOT, J1 USB_C_Receptacle_USB2.0_16P, J2 Conn_01x02_Socket, J3 Conn_01x04_Pin, J4 43045-0200, J5 Conn_01x04_Pin, U2 SN65HVD230DR, U3 USBLC6-2SC6, U4 M24C64-RMN6TP, U5 TMC2209-LA, Y1 Crystal_16MHz

Commit message: Layout Update
Parts:
- removed C4: 10uF, Capacitor_SMD:C_0402_1005Metric_Pad0.74x0.62mm_HandSolder
- removed JP1, JP2, JP3, JP4, JP5, JP6, JP7: SolderJumper_3_Open, Jumper:SolderJumper-3_P1.3mm_Open_RoundedPad1.0x1.5mm_NumberLabels
- removed JP8: SolderJumper_2_Open, Jumper:SolderJumper-2_P1.3mm_Open_RoundedPad1.0x1.5mm
- removed R13: 10k, Resistor_SMD:R_0402_1005Metric_Pad0.72x0.64mm_HandSolder
- removed R6, R7: 0R, Resistor_SMD:R_0402_1005Metric_Pad0.72x0.64mm_HandSolder
- removed S2: SKQGAKE010, KSZ_KiCad_Footprint_Library:SKQGAKE010
- removed TP1: 12V, TestPoint:TestPoint_Pad_D2.5mm
- removed TP2: 3.3V, TestPoint:TestPoint_Pad_D2.5mm
- added C34: 100nF, Capacitor_SMD:C_0402_1005Metric_Pad0.74x0.62mm_HandSolder, F.Cu at (164.2, 93.9)
- added H1: MountingHole_Pad, MountingHole:MountingHole_3.2mm_M3_ISO7380_Pad, F.Cu at (168.0, 84.8)
- added H2: MountingHole_Pad, MountingHole:MountingHole_3.2mm_M3_ISO7380_Pad, F.Cu at (137.0, 115.8)
- added H3: MountingHole_Pad, MountingHole:MountingHole_3.2mm_M3_ISO7380_Pad, F.Cu at (137.0, 84.8)
- added H4: MountingHole_Pad, MountingHole:MountingHole_3.2mm_M3_ISO7380_Pad, F.Cu at (168.0, 115.8)
- added J6: Conn_01x02_Socket, Connector_JST:JST_PH_S2B-PH-K_1x02_P2.00mm_Horizontal, F.Cu at (149.1, 118.7)
- C12, C18, C19, C20, C21, C22, C23, C24, C26, C28, C30, C32, D1, D2, D3, D4, IC2, R10, R11, R12, R17, R18, R2, R21, R24, R3, R8, R9, U4, U5: moved to B.Cu
- C27, C29: footprint Capacitor_SMD:C_0402_1005Metric_Pad0.74x0.62mm_HandSolder -> Capacitor_SMD:C_0603_1608Metric_Pad1.08x0.95mm_HandSolder
- C31, C33: value 330uF -> 10uF; footprint Capacitor_THT:CP_Radial_D6.3mm_P2.50mm -> Capacitor_SMD:C_0603_1608Metric_Pad1.08x0.95mm_HandSolder
- J2: footprint TerminalBlock:TerminalBlock_MaiXu_MX126-5.0-02P_1x02_P5.00mm -> Connector_JST:JST_PH_S2B-PH-K_1x02_P2.00mm_Horizontal
- J4: value 43045-0200 -> Conn_01x02_Socket; footprint KSZ_KiCad_Footprint_Library:43045-02YY -> Connector_JST:JST_PH_S2B-PH-K_1x02_P2.00mm_Horizontal
- S1: value SKQGAKE010 -> SKRPABE010; footprint KSZ_KiCad_Footprint_Library:SKQGAKE010 -> KSZ_KiCad_Footprint_Library:SW_SKRPABE010
- moved C31 224.6 mm to (170.2, 92.3)
- moved C33 223.8 mm to (170.2, 93.9)
- moved R22 222.7 mm to (168.5, 110.7)
- moved S1 220.2 mm to (162.7, 83.5), turned to 90 degrees
- moved R23 219.8 mm to (168.5, 89.9)
- moved J2 219.8 mm to (158.5, 118.7)
- moved J5 219.6 mm to (170.9, 103.3), turned to 90 degrees
- moved R1 219.1 mm to (163.4, 115.3)
- moved C27 215.3 mm to (170.2, 108.2)
- moved C26 212.7 mm to (168.1, 102.4), turned to -90 degrees
- moved C29 212.6 mm to (170.2, 106.7)
- moved Y1 212.4 mm to (149.9, 111.9)
- moved C21 211.9 mm to (163.6, 104.3)
- moved U3 211.4 mm to (155.2, 90.3), turned to -90 degrees
- moved C22 210.0 mm to (161.7, 105.9), turned to 90 degrees
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Connections:
- D1 pad 1: Net-(J2-Pin_2) -> /MCU_Peripherals/CANL
- D1 pad 2: Net-(J2-Pin_1) -> /MCU_Peripherals/CANH
- J2 pad 1: Net-(J2-Pin_1) -> /MCU_Peripherals/CANL
- J2 pad 2: Net-(J2-Pin_2) -> /MCU_Peripherals/CANH
- J4 pad 1: GND -> +12V
- J4 pad 2: +12V -> GND
- J5 pad 1: /Stepper_Motor_Control/B1 -> /Stepper_Motor_Control/B2
- J5 pad 2: /Stepper_Motor_Control/A1 -> /Stepper_Motor_Control/B1
- J5 pad 3: /Stepper_Motor_Control/A2 -> /Stepper_Motor_Control/A1
- J5 pad 4: /Stepper_Motor_Control/B2 -> /Stepper_Motor_Control/A2
- R5 pad 1: Net-(J2-Pin_1) -> /MCU_Peripherals/CANH
- R5 pad 2: Net-(J2-Pin_2) -> /MCU_Peripherals/CANL
- S1 pad 1: /NRST -> /U_BUTTON
- S1 pad 2: /NRST -> /U_BUTTON
- U1 pad 20: /BOOT1 -> unconnected-(U1-PB2-Pad20)
- U1 pad 21: /WC_EEPROM -> unconnected-(U1-PB10-Pad21)
- U1 pad 39: unconnected-(U1-PB3-Pad39) -> /WC_EEPROM
- U1 pad 44: /BOOT0 -> GND
- U2 pad 6: Net-(J2-Pin_2) -> /MCU_Peripherals/CANL
- U2 pad 7: Net-(J2-Pin_1) -> /MCU_Peripherals/CANH
- U3 pad 4: /MCU_Peripherals/USB1_D+ -> /USB0_D+
- U3 pad 6: /MCU_Peripherals/USB1_D- -> /USB0_D-
- U4 pad 1: /MCU_Peripherals/E0 -> GND
- U4 pad 2: /MCU_Peripherals/E1 -> GND
- U4 pad 3: /MCU_Peripherals/E2 -> GND
- U5 pad 10: Net-(JP7-C) -> GND
- U5 pad 11: Net-(JP8-A) -> /DIAG
- U5 pad 9: Net-(JP6-C) -> GND
Other:
- board outline added: 42.3 x 42.3 mm
- copper layers 2 -> 4

Commit message: Layout Update
Parts:
- D1: moved to F.Cu
- moved J6 10.4 mm to (159.5, 118.7)
- moved R5 10.3 mm to (160.5, 116.3), turned to 0 degrees
- moved J2 9.80 mm to (148.7, 118.7)
- moved D1 6.09 mm to (149.7, 115.2)
- moved R24 6.04 mm to (157.3, 104.5)
- moved C5 6.02 mm to (158.2, 89.9), turned to 0 degrees
- moved R12 4.98 mm to (145.0, 103.1), turned to 90 degrees
- moved C11 3.48 mm to (154.5, 110.7), turned to -90 degrees
- moved C23 2.97 mm to (161.2, 97.3), turned to 90 degrees
- moved C1 2.87 mm to (146.6, 103.2), turned to 90 degrees
- moved C24 2.74 mm to (160.3, 103.1)
- moved C2 2.63 mm to (149.7, 94.4), turned to 0 degrees
- moved U3 2.04 mm to (153.4, 91.3), turned to -110 degrees
- moved U2 1.81 mm to (158.1, 111.8)
- moved Y1 1.69 mm to (151.2, 110.8)
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Connections:
- D1 pad 1: /MCU_Peripherals/CANL -> /MCU_Peripherals/CAN_N
- D1 pad 2: /MCU_Peripherals/CANH -> /MCU_Peripherals/CAN_P
- J2 pad 1: /MCU_Peripherals/CANL -> /MCU_Peripherals/CAN_N
- J2 pad 2: /MCU_Peripherals/CANH -> /MCU_Peripherals/CAN_P
- J4 pad 1: +12V -> GND
- J4 pad 2: GND -> +12V
- J6 pad 1: /MCU_Peripherals/CANL -> /MCU_Peripherals/CAN_P
- J6 pad 2: /MCU_Peripherals/CANH -> /MCU_Peripherals/CAN_N
- R5 pad 1: /MCU_Peripherals/CANH -> /MCU_Peripherals/CAN_P
- R5 pad 2: /MCU_Peripherals/CANL -> /MCU_Peripherals/CAN_N
- U1 pad 26: /G_LED -> unconnected-(U1-PB13-Pad26)
- U1 pad 27: /B_LED -> /U_BUTTON
- U1 pad 28: /R_LED -> unconnected-(U1-PB15-Pad28)
- U1 pad 38: unconnected-(U1-PA15-Pad38) -> /WC_EEPROM
- U1 pad 39: /WC_EEPROM -> /R_LED
- U1 pad 40: unconnected-(U1-PB4-Pad40) -> /B_LED
- U1 pad 41: unconnected-(U1-PB5-Pad41) -> /G_LED
- U1 pad 46: /U_BUTTON -> unconnected-(U1-PB9-Pad46)
- U2 pad 6: /MCU_Peripherals/CANL -> /MCU_Peripherals/CAN_N
- U2 pad 7: /MCU_Peripherals/CANH -> /MCU_Peripherals/CAN_P
Routing:
- net /MCU_Peripherals/CAN_N: track 0.00 -> 33.8 mm
- net /MCU_Peripherals/CAN_P: track 0.00 -> 30.4 mm
- net +3.3V: track 0.00 -> 27.9 mm, vias 0 -> 6
- net /SWDIO: track 0.00 -> 26.4 mm, vias 0 -> 1
- net /SCL: track 0.00 -> 22.7 mm, vias 0 -> 2
- net /SWCLK: track 0.00 -> 22.5 mm, vias 0 -> 1
- net Net-(U5-BRA): track 0.00 -> 21.8 mm, vias 0 -> 4
- net Net-(U5-BRB): track 0.00 -> 21.5 mm, vias 0 -> 4
- net /U_BUTTON: track 0.00 -> 20.5 mm
- net /SDA: track 0.00 -> 20.5 mm, vias 0 -> 2
- net /CAN_TX: track 0.00 -> 19.5 mm, vias 0 -> 2
- net Net-(U3-VBUS): track 0.00 -> 18.2 mm
- net /CAN_RX: track 0.00 -> 16.1 mm, vias 0 -> 2
- net GND: track 0.00 -> 15.1 mm
- net /G_LED: track 0.00 -> 15.1 mm, vias 0 -> 1
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- added copper zone on B.Cu, net +12V
- added copper zone on F.Cu, net +12V
- added copper zone on B.Cu, net +3.3V
- added copper zone on F.Cu, net +3.3V
- added copper zone on B.Cu, net /Stepper_Motor_Control/A1
- added copper zone on F.Cu, net /Stepper_Motor_Control/A1
- added copper zone on B.Cu, net /Stepper_Motor_Control/A2
- added copper zone on F.Cu, net /Stepper_Motor_Control/A2
- added copper zone on B.Cu, net /Stepper_Motor_Control/B1
- added copper zone on F.Cu, net /Stepper_Motor_Control/B1
- added copper zone on B.Cu, net /Stepper_Motor_Control/B2
- added copper zone on F.Cu, net /Stepper_Motor_Control/B2
- added copper zone on B.Cu, net GND
- added copper zone on F.Cu, net GND
- added copper zone on B.Cu, net Net-(U5-BRA)
- added copper zone on F.Cu, net Net-(U5-BRA)
- added copper zone on B.Cu, net Net-(U5-BRB)
- added copper zone on F.Cu, net Net-(U5-BRB)
Other:
- board text added: "PCB_STACKUP: JLC04161H-3313"
