File: _autosave-STM32F103C8T6_FOC.kicad_pcb (KiCad board)
At the start: 4 copper layers, 42.3 x 42.3 mm, 80 parts, among them IC1 BD9E303EFJ-LBE2, IC2 AS5600-ASOT, J1 USB_C_Receptacle_USB2.0_16P, J2 Conn_01x02_Socket, J3 Conn_01x04_Pin, J4 Conn_01x02_Socket, J5 Conn_01x04_Pin, J6 Conn_01x02_Socket, U2 SN65HVD230DR, U3 USBLC6-2SC6, U4 M24C64-RMN6TP, U5 TMC2209-LA, Y1 Crystal_16MHz

Commit message: Layout Update
Routing:
- net GND: vias 104 -> 103
Changed lines of the file:
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@@
 	)
 	(via
-		(at 168.783 100.33)
-		(size 0.6)
-		(drill 0.3)
-		(layers "F.Cu" "B.Cu")
-		(free yes)
-		(net 2)
-	)
-	(via
 		(at 162.941 99.695)
 		(size 0.6)
@@
 		(polygon
 			(pts
-				(xy 165.481 98.552) (xy 167.005 99.441) (xy 167.894 99.568) (xy 167.894 100.965) (xy 167.005 101.092)
+				(xy 165.481 98.552) (xy 167.005 99.441) (xy 167.005 99.568) (xy 167.005 100.965) (xy 167.005 101.092)
 				(xy 165.481 102.108) (xy 164.719 104.14) (xy 164.719 107.188) (xy 161.163 107.188) (xy 160.909 104.267)
 				(xy 160.909 96.266) (xy 161.163 93.599) (xy 164.719 93.599) (xy 164.719 96.774)
