File: Hardware/STM32F103C8T6_FOC.kicad_pcb (KiCad board)
At the start: 4 copper layers, 42.3 x 42.3 mm, 80 parts, among them IC1 BD9E303EFJ-LBE2, IC2 AS5600-ASOT, J1 USB_C_Receptacle_USB2.0_16P, J2 Conn_01x02_Socket, J3 Conn_01x04_Pin, J4 Conn_01x02_Socket, J5 Conn_01x04_Pin, J6 Conn_01x02_Socket, U2 SN65HVD230DR, U3 USBLC6-2SC6, U4 M24C64-RMN6TP, U5 TMC2209-LA, Y1 Crystal_16MHz

Commit message: Heatsink Fix
Parts:
- moved C22 0.49 mm to (160.8, 105.4)
Routing:
- net GND: vias 98 -> 101
Changed lines of the file:
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@@
 	(footprint "Capacitor_SMD:C_0402_1005Metric_Pad0.74x0.62mm_HandSolder"
 		(layer "B.Cu")
-		(at 161.29 105.41 90)
+		(at 160.797 105.4 90)
 		(descr "Capacitor SMD 0402 (1005 Metric), square (rectangular) end terminal, IPC_7351 nominal with elongated pad for handsoldering. (Body size source: IPC-SM-782 page 76, https://www.pcb-3d.com/wordpress/wp-content/uploads/ipc-sm-782a_amendment_1_and_2.pdf), generated with kicad-footprint-generator")
 		(tags "capacitor handsolder")
@@
 	)
 	(via
-		(at 165.1 98.933)
+		(at 152.4508 93.990499)
 		(size 0.6)
 		(drill 0.3)
 		(layers "F.Cu" "B.Cu")
+		(free yes)
 		(net 2)
 	)
 	(via
-		(at 152.4508 93.990499)
+		(at 158.402009 92.881101)
 		(size 0.6)
 		(drill 0.3)
@@
 	)
 	(via
-		(at 158.402009 92.881101)
+		(at 164.497 104.7634)
 		(size 0.6)
 		(drill 0.3)
@@
 	)
 	(via
-		(at 162.941 101.092)
+		(at 135.6614 108.9152)
 		(size 0.6)
 		(drill 0.3)
 		(layers "F.Cu" "B.Cu")
+		(free yes)
 		(net 2)
 	)
 	(via
-		(at 135.6614 108.9152)
+		(at 155.321 105.7656)
 		(size 0.6)
 		(drill 0.3)
@@
 	)
 	(via
-		(at 155.321 105.7656)
+		(at 158.3182 103.6828)
 		(size 0.6)
 		(drill 0.3)
@@
 	)
 	(via
-		(at 158.3182 103.6828)
+		(at 163.267 96.92)
 		(size 0.6)
 		(drill 0.3)
@@
 	)
 	(via
-		(at 163.703 98.933)
+		(at 162.427 93.9)
 		(size 0.6)
 		(drill 0.3)
 		(layers "F.Cu" "B.Cu")
+		(free yes)
 		(net 2)
 	)
@@
 	)
 	(via
-		(at 143.383 106.5276)
+		(at 161.597 104.97)
 		(size 0.6)
 		(drill 0.3)
@@
 	)
 	(via
-		(at 164.465 99.695)
+		(at 143.383 106.5276)
 		(size 0.6)
 		(drill 0.3)
 		(layers "F.Cu" "B.Cu")
+		(free yes)
 		(net 2)
 	)
 	(via
-		(at 134.6962 93.472)
+		(at 134.737 93.08)
 		(size 0.6)
 		(drill 0.3)
@@
 	)
 	(via
+		(at 163.427 94.78)
+		(size 0.6)
+		(drill 0.3)
+		(layers "F.Cu" "B.Cu")
+		(free yes)
+		(net 2)
+	)
+	(via
 		(at 151.7142 97.5868)
 		(size 0.6)
@@
 	)
 	(via
+		(at 161.667 105.6)
+		(size 0.6)
+		(drill 0.3)
+		(layers "F.Cu" "B.Cu")
+		(free yes)
+		(net 2)
+	)
+	(via
 		(at 144.2466 101.7016)
 		(size 0.6)
@@
 	)
 	(via
-		(at 162.306 98.933)
+		(at 161.747 104.31)
 		(size 0.6)
 		(drill 0.3)
 		(layers "F.Cu" "B.Cu")
+		(free yes)
 		(net 2)
 	)
@@
 	)
 	(via
-		(at 165.1 100.33)
-		(size 0.6)
-		(drill 0.3)
-		(layers "F.Cu" "B.Cu")
-		(net 2)
-	)
-	(via
 		(at 154.9908 119.0498)
 		(size 0.6)
@@
 	)
 	(via
-		(at 162.306 101.727)
-		(size 0.6)
-		(drill 0.3)
-		(layers "F.Cu" "B.Cu")
-		(net 2)
-	)
-	(via
 		(at 159.279417 107.933107)
 		(size 0.6)
@@
 	)
 	(via
-		(at 163.687 100.33)
+		(at 161.544 102.489)
 		(size 0.6)
 		(drill 0.3)
 		(layers "F.Cu" "B.Cu")
+		(free yes)
 		(net 2)
 	)
 	(via
-		(at 161.544 102.489)
+		(at 160.2994 99.6696)
 		(size 0.6)
 		(drill 0.3)
@@
 	)
 	(via
-		(at 160.2994 99.6696)
+		(at 159.687 104.56)
 		(size 0.6)
 		(drill 0.3)
@@
 	)
 	(via
-		(at 159.385 104.9528)
+		(at 147.197 101.1594)
 		(size 0.6)
 		(drill 0.3)
@@
 	)
 	(via
-		(at 165.1 101.727)
+		(at 158.877 97.8408)
 		(size 0.6)
 		(drill 0.3)
 		(layers "F.Cu" "B.Cu")
+		(free yes)
 		(net 2)
 	)
 	(via
-		(at 147.197 101.1594)
+		(at 142.2654 102.5144)
 		(size 0.6)
 		(drill 0.3)
@@
 	)
 	(via
-		(at 158.877 97.8408)
+		(at 142.8496 96.0374)
 		(size 0.6)
 		(drill 0.3)
@@
 	)
 	(via
-		(at 142.2654 102.5144)
+		(at 164.257 93.91)
 		(size 0.6)
 		(drill 0.3)
@@
 	)
 	(via
-		(at 142.8496 96.0374)
+		(at 152.273 89.027)
 		(size 0.6)
 		(drill 0.3)
@@
 	)
 	(via
-		(at 152.273 89.027)
+		(at 156.083 88.6714)
 		(size 0.6)
 		(drill 0.3)
@@
 	)
 	(via
-		(at 156.083 88.6714)
+		(at 161.5694 120.5992)
 		(size 0.6)
 		(drill 0.3)
@@
 	)
 	(via
-		(at 161.5694 120.5992)
+		(at 161.977 96.83)
 		(size 0.6)
 		(drill 0.3)
@@
 	)
 	(via
-		(at 162.941 99.695)
+		(at 162.363353 105.535)
 		(size 0.6)
 		(drill 0.3)
 		(layers "F.Cu" "B.Cu")
+		(free yes)
 		(net 2)
 	)
@@
 	)
 	(via
-		(at 164.465 101.092)
+		(at 161.407 94.85)
 		(size 0.6)
 		(drill 0.3)
 		(layers "F.Cu" "B.Cu")
+		(free yes)
 		(net 2)
 	)
@@
 	)
 	(via
+		(at 161.627676 106.270676)
+		(size 0.6)
+		(drill 0.3)
+		(layers "F.Cu" "B.Cu")
+		(free yes)
+		(net 2)
+	)
+	(via
 		(at 154.283454 94.432597)
 		(size 0.6)
@@
 	)
 	(via
+		(at 159.627 101.6)
+		(size 0.6)
+		(drill 0.3)
+		(layers "F.Cu" "B.Cu")
+		(free yes)
+		(net 2)
+	)
+	(via
 		(at 155.4226 113.9444)
 		(size 0.6)
@@
 	)
 	(via
-		(at 163.703 101.727)
+		(at 164.417 103.63)
 		(size 0.6)
 		(drill 0.3)
 		(layers "F.Cu" "B.Cu")
+		(free yes)
 		(net 2)
 	)
@@
 	)
 	(via
-		(at 160.4772 106.4514)
+		(at 159.707 105.32)
 		(size 0.6)
 		(drill 0.3)
@@
 	)
 	(via
-		(at 162.306 100.33)
+		(at 154.4574 108.3564)
 		(size 0.6)
 		(drill 0.3)
 		(layers "F.Cu" "B.Cu")
+		(free yes)
 		(net 2)
 	)
 	(via
-		(at 154.4574 108.3564)
+		(at 147.3962 115.1128)
 		(size 0.6)
 		(drill 0.3)
@@
 	)
 	(via
-		(at 147.3962 115.1128)
+		(at 156.845 95.7072)
 		(size 0.6)
 		(drill 0.3)
@@
 	)
 	(via
-		(at 156.845 95.7072)
+		(at 161.077 103.15)
 		(size 0.6)
 		(drill 0.3)
@@
 		(net 2)
 	)
+	(via
+		(at 163.387 94.01)
+		(size 0.6)
+		(drill 0.3)
+		(layers "F.Cu" "B.Cu")
+		(free yes)
+		(net 2)
+	)
 	(segment
 		(start 161.237 99.33)
@@
 	)
 	(segment
-		(start 161.29 107.188)
-		(end 161.29 105.9775)
+		(start 160.797 106.695)
+		(end 160.797 106.0875)
 		(width 0.5)
 		(layer "B.Cu")
@@
 	(segment
 		(start 162.687 108.585)
-		(end 161.29 107.188)
+		(end 160.797 106.695)
 		(width 0.5)
 		(layer "B.Cu")
@@
 	)
 	(segment
-		(start 161.544 103.632)
-		(end 161.29 103.886)
+		(start 162.687 103.291838)
+		(end 162.346838 103.632)
 		(width 0.3)
 		(layer "B.Cu")
@@
 	)
 	(segment
-		(start 162.346838 103.632)
-		(end 161.544 103.632)
+		(start 162.687 102.78)
+		(end 162.687 103.291838)
 		(width 0.3)
 		(layer "B.Cu")
@@
 	)
 	(segment
-		(start 162.687 102.78)
-		(end 162.687 103.291838)
+		(start 162.346838 103.632)
+		(end 161.544 103.632)
 		(width 0.3)
 		(layer "B.Cu")
@@
 	)
 	(segment
-		(start 162.687 103.291838)
-		(end 162.346838 103.632)
+		(start 161.544 103.632)
+		(end 160.797 104.379)
 		(width 0.3)
 		(layer "B.Cu")
@@
 	)
 	(segment
-		(start 161.29 103.886)
-		(end 161.29 104.8425)
+		(start 160.797 104.379)
+		(end 160.797 104.8325)
 		(width 0.3)
 		(layer "B.Cu")
@@
 	)
 	(segment
-		(start 163.195 96.4692)
-		(end 164.187 97.4612)
+		(start 160.3502 93.8784)
+		(end 161.3662 93.8784)
 		(width 0.2)
 		(layer "B.Cu")
@@
 	)
 	(segment
-		(start 160.3502 93.8784)
-		(end 161.3662 93.8784)
+		(start 164.187 97.06029)
+		(end 164.187 97.88)
 		(width 0.2)
 		(layer "B.Cu")
@@
 	)
 	(segment
-		(start 164.187 97.4612)
-		(end 164.187 97.88)
+		(start 161.3662 93.8784)
+		(end 163.641 96.1532)
 		(width 0.2)
 		(layer "B.Cu")
@@
 	)
 	(segment
-		(start 163.195 95.7072)
-		(end 163.195 96.4692)
+		(start 163.641 96.1532)
+		(end 163.641 96.51429)
 		(width 0.2)
 		(layer "B.Cu")
@@
 	)
 	(segment
-		(start 161.3662 93.8784)
-		(end 163.195 95.7072)
+		(start 163.641 96.51429)
+		(end 164.187 97.06029)
 		(width 0.2)
 		(layer "B.Cu")
